Commit message: Driving the Virtual Robot

File: description/robot.urdf.xacro (robot description, xacro)
@@ -2,3 +2,4 @@
 <robot xmlns:xacro="http://www.ros.org/wiki/xacro"  name="robot">
     <xacro:include filename="rover_core.xacro" />
+    <xacro:include filename="rover_control.xacro" />
 </robot>

File: description/rover_core.xacro (robot description, xacro)
@@ -40,4 +40,7 @@
 	    </xacro:inertial_box>
 	</link>
+	<gazebo reference="chassis">
+		<material>Gazebo/White</material>
+	</gazebo>
 	<!-- LEFT WHEEL -->
 	<joint name="left_wheel_joint" type="continuous">
@@ -63,4 +66,7 @@
 	    </xacro:inertial_cylinder>
 	</link>
+	<gazebo reference="left_wheel">
+		<material>Gazebo/Blue</material>
+	</gazebo>
 	<!-- RIGHT WHEEL -->
 	<joint name="right_wheel_joint" type="continuous">
@@ -86,4 +92,7 @@
 	    </xacro:inertial_cylinder>
 	</link>
+	<gazebo reference="right_wheel">
+		<material>Gazebo/Blue</material>
+	</gazebo>
 	<!-- CASTER WHEEL -->
 	<joint name="caster_wheel_joint" type="fixed">
@@ -108,3 +117,8 @@
 	    </xacro:inertial_sphere>
 	</link>
+	<gazebo reference="caster_wheel">
+		<material>Gazebo/Black</material>
+		<mu1 value="0.0001"/>
+		<mu2 value="0.0001"/>
+	</gazebo>
 </robot>
