Commit message: Added Realsense Moule [Gazebo and URDF]

File: description/robot.urdf.xacro (robot description, xacro)
@@ -2,9 +2,86 @@
 <robot xmlns:xacro="http://www.ros.org/wiki/xacro"  name="robot">
     <xacro:include filename="robot_base1.xacro" />
-    <xacro:include filename="lidar1.xacro" />
+    <!-- <xacro:include filename="lidar1.xacro" /> -->
     <!-- <xacro:include filename="ros2_control.xacro" /> -->
     <!-- <xacro:include filename="3d_lidar1.xacro" /> -->
-    <xacro:include filename="camera.xacro" />
+    <!-- <xacro:include filename="camera.xacro" /> -->
     <!-- <xacro:include filename="depth_camera.xacro" /> -->
-    <xacro:include filename="gazebo_control1.xacro" />
+    <!-- <xacro:include filename="gazebo_control1.xacro" /> -->
+    <!-- <xacro:include filename="realsence.xacro" /> -->
+    <link name="camera_bottom_screw_frame">
+    <visual>
+      <geometry>
+        <mesh filename="package://chiconybot_description/meshes/sensors/d435.dae" />
+      </geometry>
+    </visual>
+    <collision>
+      <geometry>
+        <mesh filename="package://chiconybot_description/meshes/sensors/d435.dae" />
+      </geometry>
+    </collision>
+  </link>
+  <link name="camera_link"></link>
+  <link name="camera_depth_frame"></link>
+  <link name="camera_depth_optical_frame"></link>
+  <link name="camera_color_frame"></link>
+  <link name="camera_color_optical_frame"></link>
+  <link name="camera_left_ir_frame"></link>
+  <link name="camera_left_ir_optical_frame"></link>
+  <link name="camera_right_ir_frame"></link>
+  <link name="camera_right_ir_optical_frame"></link>
+   <joint name="camera_joint" type="fixed">
+    <parent link="base_link" />
+    <child link="camera_bottom_screw_frame" />
+    <pose xyz="0.4 0 0.25" rpy="0 0 0" />
+  </joint>
+  <joint name="camera_link_joint" type="fixed">
+    <parent link="camera_bottom_screw_frame" />
+    <child link="camera_link" />
+    <pose xyz="0 0.0175 0.0125 " rpy="0 0 0" />
+  </joint>
+  <joint name="camera_depth_joint" type="fixed">
+    <parent link="camera_link" />
+    <child link="camera_depth_frame" />
+    <pose xyz="0 0 0" rpy="0 0 0" />
+  </joint>
+  <joint name="camera_depth_optical_joint" type="fixed">
+    <parent link="camera_depth_frame" />
+    <child link="camera_depth_optical_frame" />
+    <pose xyz="0 0 0 " rpy="-1.57 0 -1.57" />
+  </joint>
+  <joint name="camera_color_joint" type="fixed">
+    <parent link="camera_depth_frame" />
+    <child link="camera_color_frame" />
+    <pose xyz="0 0 0" rpy="0 0 0" />
+  </joint>
+  <joint name="camera_color_optical_joint" type="fixed">
+    <parent link="camera_color_frame" />
+    <child link="camera_color_optical_frame" />
+    <pose xyz="0 0 0 " rpy="-1.57 0 -1.57" />
+  </joint>
+  <joint name="camera_left_ir_joint" type="fixed">
+    <parent link="camera_depth_frame" />
+    <child link="camera_left_ir_frame" />
+    <pose xyz="0 0 0 " rpy="0 0 0 " />
+  </joint>
+  <joint name="camera_left_ir_optical_joint" type="fixed">
+    <parent link="camera_left_ir_frame" />
+    <child link="camera_left_ir_optical_frame" />
+    <pose xyz="0 0 0 " rpy="-1.57 0 -1.57" />
+  </joint>
+  <joint name="camera_right_ir_joint" type="fixed">
+    <parent link="camera_depth_frame" />
+    <child link="camera_right_ir_frame" />
+    <pose xyz="0 -0.050 0 " rpy="0 0 0" />
+  </joint>
+  <joint name="camera_right_ir_optical_joint" type="fixed">
+    <parent link="camera_right_ir_frame" />
+    <child link="camera_right_ir_optical_frame" />
+    <pose xyz="0 0 0 " rpy="-1.57 0 -1.57" />
+  </joint>
+    <gazebo>
+        <include>
+            <uri>model://realsense_model</uri>
+        </include>
+    </gazebo>
 </robot>
