Commit message: Before Changes made to make perfecr rover

File: description/gazebo_control.xacro (robot description, xacro)
@@ -1,21 +1,25 @@
 <?xml version="1.0"?>
-<robot xmlns:xacro="http://www.ros.org/wiki/xacro">
-    <gazebo>
-        <plugin name="diff_drive" filename="libgazebo_ros_diff_drive.so">
-            <!-- Wheel Information -->
-            <left_joint>left_wheel_joint</left_joint>
-            <right_joint>right_wheel_joint</right_joint>
-            <wheel_separation>0.35</wheel_separation>
-            <wheel_diameter>0.1</wheel_diameter>
-            <!-- Limits -->
-            <max_wheel_torque>200</max_wheel_torque>
-            <max_wheel_acceleration>10.0</max_wheel_acceleration>
-            <!-- Output -->
-            <odometry_frame>odom</odometry_frame>
-            <robot_base_frame>base_link</robot_base_frame>
-            <publish_odom>true</publish_odom>
-            <publish_odom_tf>true</publish_odom_tf>
-            <publish_wheel_tf>true</publish_wheel_tf>
-        </plugin>
+<robot xmlns:xacro="http://www.ros.org/wiki/xacro" >
+	<gazebo>
+		<plugin name='wheel_drive_controller' filename='libgazebo_ros_diff_drive_mod.so'>
+			<!-- wheels -->
+			<num_wheel_pairs>2</num_wheel_pairs>
+            <left_joint>front_left_joint</left_joint>
+            <left_joint>back_left_joint</left_joint>
+            <right_joint>front_right_joint</right_joint>
+            <right_joint>back_right_joint</right_joint>
+			<!-- kinematics -->
+			<wheel_separation>0.35</wheel_separation>
+			<wheel_diameter>0.1</wheel_diameter>
+			<!-- limits -->
+			<max_wheel_torque>100</max_wheel_torque>
+			<max_wheel_acceleration>10</max_wheel_acceleration>
+			<!-- output -->
+			<publish_odom>true</publish_odom>
+			<publish_odom_tf>true</publish_odom_tf>
+			<publish_wheel_tf>true</publish_wheel_tf>
+			<odometry_frame>odom</odometry_frame>
+			<robot_base_frame>base_link</robot_base_frame>
+		</plugin>
     </gazebo>
 </robot>

File: description/lidar1.xacro (robot description, xacro)
@@ -1,22 +1,22 @@
 <?xml version="1.0"?>
-<robot xmlns:xacro="http://www.ros.org/wiki/xacro" >
+<robot xmlns:xacro="http://www.ros.org/wiki/xacro">
     <joint name="laser_joint" type="fixed">
         <parent link="chassis"/>
         <child link="laser_frame"/>
-        <origin xyz="0.2 0.0 0.12" rpy="0 0 ${-pi}"/>
+        <origin xyz="0.3 0 0.21" rpy="0 0 0"/>
     </joint>
     <link name="laser_frame">
         <visual>
             <geometry>
-                <cylinder radius="0.05" length="0.04"/>
+                <cylinder radius="0.05" length="0.04" />
             </geometry>
-            <material name="orange"/>
+            <material name="white" />
         </visual>
         <collision>
             <geometry>
-                <cylinder radius="0.05" length="0.04"/>
+                <cylinder radius="0.05" length="0.04" />
             </geometry>
         </collision>
-        <xacro:inertial_cylinder mass="0.1" length="0.04" radius="0.05" >
+        <xacro:inertial_cylinder mass="0.1" length="0.04" radius="0.05">
             <origin xyz="0 0 0" rpy="0 0 0"/>
         </xacro:inertial_cylinder>
@@ -24,7 +24,7 @@
     <!-- Sensor ray -->
     <gazebo reference="laser_frame">
-        <material>Gazebo/Orange</material>
-        <sensor name="laser" type="ray" >
-            <pose>0 0 0 0 0 0</pose>
+        <material>Gazebo/White</material>
+        <sensor name="laser" type="ray">
+            <pose>0 0 0 0 0 0 </pose>
             <update_rate>10</update_rate>
             <visualize>true</visualize>
@@ -39,10 +39,10 @@
                 </scan>
                 <range>
-                    <min>0.5</min>
-                    <max>10</max>
+                    <min>0.3</min>
+                    <max>12</max>
                     <resolution>0.01</resolution>
                 </range>
             </ray>
-            <plugin name="laser_controller" filename="libgazebo_ros_ray_sensor.so" >
+            <plugin name="laser_controller" filename="libgazebo_ros_ray_sensor.so">
                 <ros>
                     <argument>~/out:=scan</argument>

File: description/robot.urdf.xacro (robot description, xacro)
@@ -1,9 +1,10 @@
 <?xml version="1.0"?>
 <robot xmlns:xacro="http://www.ros.org/wiki/xacro"  name="robot">
-    <xacro:include filename="robot_base.xacro" />
-    <xacro:include filename="lidar.xacro" />
-    <!-- <xacro:include filename="camera.xacro" /> -->
-    <xacro:include filename="depth_camera.xacro" />
-    <xacro:include filename="gazebo_control.xacro" />
+    <xacro:include filename="robot_base1.xacro" />
+    <xacro:include filename="lidar1.xacro" />
     <!-- <xacro:include filename="ros2_control.xacro" /> -->
+    <!-- <xacro:include filename="3d_lidar1.xacro" /> -->
+    <xacro:include filename="camera.xacro" />
+    <!-- <xacro:include filename="depth_camera.xacro" /> -->
+    <xacro:include filename="gazebo_control1.xacro" />
 </robot>

File: description/robot_base.xacro (robot description, xacro)
@@ -1,21 +1,22 @@
 <?xml version="1.0"?>
 <robot xmlns:xacro="http://www.ros.org/wiki/xacro" >
-    <xacro:include filename="inertial_macros.xacro" />
+    <xacro:include filename="inertial_macros.xacro"/>
+    <!-- COLORS -->
     <material name="white">
-        <color rgba="1 1 1 1"/>
+        <color rgba="1 1 1 1.0"/>
+    </material>
+    <material name="orange">
+        <color rgba="1 0.3 .1 1.0"/>
     </material>
     <material name="blue">
-        <color rgba="1 0.3 0.1 1"/>
+        <color rgba=".2 .2 1 1.0"/>
+    </material>
+    <material name="black">
+        <color rgba="0 0 0 1.0"/>
     </material>
     <material name="blurrywood">
         <color rgba="1 0.4 0.2 1"/>
     </material>
-    <material name="black">
-        <color rgba="0 0 0 1"/>
-    </material>
-    <material name="orange">
-        <color rgba="1 0.3 0.1 1"/>
-    </material>
-    <!--BASE LINK-->
+    <!-- Base_Link-->
     <link name="base_link">
     </link>
@@ -28,148 +29,139 @@
     <link name="base_footprint">
     </link>
-    <!--CHASSIS LINK-->
+    <!-- Chassis-->
     <joint name="chassis_joint" type="fixed">
         <parent link="base_link"/>
         <child link="chassis"/>
-        <origin xyz="-0.1 0 0"/>
+        <origin xyz="0.0 0.0 0.0" rpy="0.0 0.0 0.0"/>
     </joint>
     <link name="chassis">
         <visual>
-            <origin xyz="0.25 0 0.1" />
+            <origin xyz="0.0 0.0 0.05"/>
             <geometry>
-                <box size="0.5 0.3 0.2" />
-            </geometry>oo
-            <material name="blurrywood" />
+                <box size="0.4 .3 .1"/>
+            </geometry>
+            <material name="white"/>
         </visual>
         <collision>
-            <origin xyz="0.25 0 0.1" />
+            <origin xyz="0.0 0.0 0.05"/>
             <geometry>
-                <box size="0.5 0.3 0.2" />
+                <box size=".4 .3 .1"/>
             </geometry>
         </collision>
-        <xacro:inertial_box mass="0.5" x="0.5" y="0.3" z="0.2">
-            <origin xyz="0.25 0 0.1" rpy="0 0 0"/>
+        <xacro:inertial_box mass="0.5" x="0.4" y="0.3" z="0.1">
+            <origin xyz="0.0 0.0 0.5"/>
         </xacro:inertial_box>
     </link>
     <gazebo reference="chassis">
-        <material>
-            Gazebo/Orange
-        </material>
+        <material>Gazebo/White</material>
     </gazebo>
-    <!-- LEFT WHEEL LINK-->
-    <joint name="left_wheel_joint" type="continuous">
-        <parent link="base_link" />
-        <child link="left_wheel" />
-        <origin xyz="0 0.175 0" rpy="-${pi/2} 0 0" />
-        <axis xyz="0 0 1"/>
+    <!-- WHEELS -->
+    <joint name="front_left_joint" type="continuous" >
+        <origin xyz="0.15 .175 0.0" rpy="${-pi/2} 0.0 0.0"/>
+        <parent link="base_link"/>
+        <child link="left_front_wheel"/>
+        <axis xyz="0.0 0.0 1"/>
     </joint>
-    <link name="left_wheel">
+    <link name="left_front_wheel">
         <visual>
             <geometry>
-                <cylinder radius="0.05" length="0.04" />
+                <cylinder radius=".05" length=".04"/>
             </geometry>
-            <material name="black" />
+            <material name="blue"/>
         </visual>
         <collision>
             <geometry>
-                <sphere radius="0.05" />
+                <cylinder radius=".05" length=".04"/>
             </geometry>
         </collision>
-        <xacro:inertial_cylinder mass="0.1" length="0.04" radius="0.05">
-            <origin xyz="0 0 0" rpy="0 0 0"/>
+        <xacro:inertial_cylinder mass="0.1" radius=".05" length=".04">
+            <origin xyz="0.0 0.0 0.5"/>
         </xacro:inertial_cylinder>
     </link>
-    <gazebo reference="left_wheel">
-        <material>
-            Gazebo/Black
-        </material>
+    <gazebo reference="left_front_wheel">
+        <material>Gazebo/Blue</material>
+        <mu1 value="0.001"/>
+        <mu2 value="0.001"/>
     </gazebo>
-    <!-- RIGHT WHEEL LINK-->
-    <joint name="right_wheel_joint" type="continuous">
-        <parent link="base_link" />
-        <child link="right_wheel" />
-        <origin xyz="0 -0.175 0" rpy="${pi/2} 0 0" />
-        <axis xyz="0 0 -1"/>
+    <joint name="front_right_joint" type="continuous" >
+        <origin xyz="0.15 -.175 0.0" rpy="${pi/2} 0.0 0.0"/>
+        <parent link="base_link"/>
+        <child link="right_front_wheel"/>
+        <axis xyz="0.0 0.0 -1"/>
     </joint>
-    <link name="right_wheel">
+    <link name="right_front_wheel">
         <visual>
             <geometry>
-                <cylinder radius="0.05" length="0.04" />
+                <cylinder radius=".05" length=".04"/>
             </geometry>
-            <material name="black" />
+            <material name="blue"/>
         </visual>
         <collision>
             <geometry>
-                <sphere radius="0.05" />
+                <cylinder radius=".05" length=".04"/>
             </geometry>
         </collision>
-        <xacro:inertial_cylinder mass="0.1" length="0.04" radius="0.05">
-            <origin xyz="0 0 0" rpy="0 0 0"/>
+        <xacro:inertial_cylinder mass="0.1" radius=".05" length=".04">
+            <origin xyz="0.0 0.0 0.5"/>
         </xacro:inertial_cylinder>
     </link>
-    <gazebo reference="right_wheel">
-        <material>
-            Gazebo/Black
-        </material>
+    <gazebo reference="right_front_wheel">
+        <material>Gazebo/Blue</material>
+        <mu1 value="0.001"/>
+        <mu2 value="0.001"/>
     </gazebo>
-    <!-- LEFT CASTER WHEELS LINK-->
-    <joint name="left_caster_wheel_joint" type="fixed">
-        <parent link="chassis" />
-        <child link="left_caster_wheel" />
-        <origin xyz="0.4 0.175 0" rpy="-${pi/2} 0 0"/>
-        <axis xyz="0 0 1"/>
+    <joint name="back_left_joint" type="continuous" >
+        <origin xyz="-0.15 .175 0.0" rpy="${-pi/2} 0.0 0.0"/>
+        <parent link="base_link"/>
+        <child link="left_back_wheel"/>
+        <axis xyz="0.0 0.0 1"/>
     </joint>
-    <link name="left_caster_wheel">
+    <link name="left_back_wheel">
         <visual>
             <geometry>
-                <cylinder radius="0.05" length="0.04"/>
+                <cylinder radius=".05" length=".04"/>
             </geometry>
-            <material name="black" />
+            <material name="black"/>
         </visual>
         <collision>
             <geometry>
-                <cylinder radius="0.05" length="0.04"/>
+                <cylinder radius=".05" length=".04"/>
             </geometry>
         </collision>
-        <xacro:inertial_cylinder mass="0.1" length="0.04" radius="0.05">
-            <origin xyz="0 0 0" rpy="0 0 0"/>
+        <xacro:inertial_cylinder mass="0.1" radius=".05" length=".04">
+            <origin xyz="0.0 0.0 0.5"/>
         </xacro:inertial_cylinder>
     </link>
-    <gazebo reference="left_caster_wheel">
-        <material>
-            Gazebo/Black
-        </material>
-        <mu1 value="0.01" />
-        <mu2 value="0.01" />
+    <gazebo reference="left_back_wheel">
+        <material>Gazebo/Black</material>
+        <mu1 value="0.001"/>
+        <mu2 value="0.001"/>
     </gazebo>
-        <!-- RIGHT CASTER WHEELS LINK-->
-        <joint name="right_caster_wheel_joint" type="fixed">
-            <parent link="chassis" />
-            <child link="right_caster_wheel" />
-            <origin xyz="0.4 -0.175 0" rpy="${pi/2} 0 0"/>
-            <axis xyz="0 0 -1"/>
-        </joint>
-        <link name="right_caster_wheel">
-            <visual>
-                <geometry>
-                    <cylinder radius="0.05" length="0.04"/>
-                </geometry>
-                <material name="black" />
-            </visual>
-            <collision>
-                <geometry>
-                    <cylinder radius="0.05" length="0.04"/>
-                </geometry>
-            </collision>
-            <xacro:inertial_cylinder mass="0.1" length="0.04" radius="0.05">
-                <origin xyz="0 0 0" rpy="0 0 0"/>
-            </xacro:inertial_cylinder>
-        </link>
-        <gazebo reference="right_caster_wheel">
-            <material>
-                Gazebo/Black
-            </material>
-            <mu1 value="0.01" />
-            <mu2 value="0.01" />
-        </gazebo>
+    <joint name="back_right_joint" type="continuous" >
+        <origin xyz="-0.15 -.175 0.0" rpy="${pi/2} 0.0 0.0"/>
+        <parent link="base_link"/>
+        <child link="right_back_wheel"/>
+        <axis xyz="0.0 0.0 -1"/>
+    </joint>
+    <link name="right_back_wheel">
+        <visual>
+            <geometry>
+                <cylinder radius=".05" length=".04"/>
+            </geometry>
+            <material name="black"/>
+        </visual>
+        <collision>
+            <geometry>
+                <cylinder radius=".05" length=".04"/>
+            </geometry>
+        </collision>
+        <xacro:inertial_cylinder mass="0.1" radius=".05" length=".04">
+            <origin xyz="0.0 0.0 0.5"/>
+        </xacro:inertial_cylinder>
+    </link>
+    <gazebo reference="right_back_wheel">
+        <material>Gazebo/Black</material>
+        <mu1 value="0.001"/>
+        <mu2 value="0.001"/>
+    </gazebo>
 </robot>

File: description/ros2_control.xacro (robot description, xacro)
@@ -5,5 +5,5 @@
             <plugin>gazebo_ros2_control/GazeboSystem</plugin>
         </hardware>
-        <joint name="left_wheel_joint">
+        <joint name="front_left_joint">
             <command_interface name="velocity">
                 <param name="min">-10</param>
@@ -13,5 +13,21 @@
             <state_interface name="position"/>
         </joint>
-        <joint name="right_wheel_joint">
+        <joint name="back_left_joint">
+            <command_interface name="velocity">
+                <param name="min">-10</param>
+                <param name="max">10</param>
+            </command_interface>
+            <state_interface name="velocity"/>
+            <state_interface name="position"/>
+        </joint>
+        <joint name="front_right_joint">
+            <command_interface name="velocity">
+                <param name="min">-10</param>
+                <param name="max">10</param>
+            </command_interface>
+            <state_interface name="velocity"/>
+            <state_interface name="position"/>
+        </joint>
+        <joint name="back_right_joint">
             <command_interface name="velocity">
                 <param name="min">-10</param>
